File: chili-audio-module-hardware.kicad_pcb (KiCad board)
At the start: 2 copper layers, 11.5 x 17.5 mm, 7 parts, among them J1 Conn_01x04_Pin, J2 Conn_01x02_Pin, J3 MX1.25_2Pin, U1 MAX98357A

Commit message: finishing touches
Parts:
- added G***: LOGO, LOGO, B.Cu at (129.0, 97.2)
- added ROHS: RoHS-Logo_6mm_SilkScreen, Symbol:RoHS-Logo_6mm_SilkScreen, B.Cu at (125.5, 95.0)
Other:
- board text added: "3V3"
- board text added: "BCLK"
- board text added: "DIN"
- board text added: "GND"
- board text added: "LRCLK"
- board text added: "MODE"
- board text added: "chili-audio-module"
- board text added: "chilichip"
- board text added: "v1.0.0"

Commit message: small correction
Parts:
- moved J2 0.41 mm to (132.5, 107.0)
Changed lines of the file:
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@@
 	(footprint "Connector_PinHeader_2.54mm:PinHeader_1x02_P2.54mm_Vertical"
 		(layer "B.Cu")
-		(at 132.09 107 90)
+		(at 132.5 107 90)
 		(descr "Through hole straight pin header, 1x02, 2.54mm pitch, single row")
 		(tags "Through hole pin header THT 1x02 2.54mm single row")
@@
 	)
 	(gr_text "GND"
-		(at 128.25 109 0)
+		(at 128.5 109 0)
 		(layer "F.SilkS")
 		(effects
@@
 	)
 	(gr_text "3V3"
-		(at 131 109 0)
+		(at 131.5 109 0)
 		(layer "F.SilkS")
 		(effects
@@
 	)
 	(segment
+		(start 134.35 101.85)
+		(end 134.35 105.15)
+		(width 0.3)
+		(layer "F.Cu")
+		(net "+3.3V")
+	)
+	(segment
+		(start 132.67 101.13)
+		(end 133.63 101.13)
+		(width 0.3)
+		(layer "F.Cu")
+		(net "+3.3V")
+	)
+	(segment
 		(start 131.5475 101.1325)
 		(end 131.5475 100.6325)
@@
 	(segment
 		(start 133.63 101.13)
-		(end 132.67 101.13)
-		(width 0.3)
-		(layer "F.Cu")
-		(net "+3.3V")
-	)
-	(segment
-		(start 132.09 107)
-		(end 134.35 104.74)
-		(width 0.3)
-		(layer "F.Cu")
-		(net "+3.3V")
-	)
-	(segment
-		(start 134.35 104.74)
 		(end 134.35 101.85)
 		(width 0.3)
@@
 	)
 	(segment
-		(start 134.35 101.85)
-		(end 133.63 101.13)
-		(width 0.3)
-		(layer "F.Cu")
+		(start 134.35 105.15)
+		(end 132.5 107)
+		(width 0.3)
+		(layer "F.Cu")
